Commit message: add mujoco visualizer

File: assets/allegro/allegro_internal_mujoco.urdf (robot description, URDF)
Before this commit: robot allegro_hand_right, 21 links, 20 joints
Links:
- link base_link: geometry collision box size=0.01 0.01 0.01; visual mesh filename=base_link.obj
- link link_0.0: geometry collision box size=0.0196 0.0275 0.0164; visual mesh filename=link_0.0.obj
- link link_1.0: geometry collision box size=0.0196 0.0275 0.054; visual mesh filename=link_1.0.obj
- link link_10.0: geometry collision box size=0.0196 0.0275 0.0384; visual mesh filename=link_2.0.obj
- link link_11.0: geometry collision sphere radius=0.0001; visual mesh filename=link_3.0.obj
- link link_12.0: geometry collision box size=0.0358 0.034 0.0455; visual mesh filename=link_12.0_right.obj
- link link_13.0: geometry collision box size=0.0196 0.0275 0.0177; visual mesh filename=link_13.0.obj
- link link_14.0: geometry collision box size=0.0196 0.0275 0.0514; visual mesh filename=link_14.0.obj
- link link_15.0: geometry collision sphere radius=0.0001; visual mesh filename=link_15.0.obj
- link link_2.0: geometry collision box size=0.0196 0.0275 0.0384; visual mesh filename=link_2.0.obj
- link link_3.0: geometry collision sphere radius=0.0001; visual mesh filename=link_3.0.obj
- link link_4.0: geometry collision box size=0.0196 0.0275 0.0164; visual mesh filename=link_0.0.obj
- link link_5.0: geometry collision box size=0.0196 0.0275 0.054; visual mesh filename=link_1.0.obj
- link link_6.0: geometry collision box size=0.0196 0.0275 0.0384; visual mesh filename=link_2.0.obj
- link link_7.0: geometry collision sphere radius=0.0001; visual mesh filename=link_3.0.obj
- link link_8.0: geometry collision box size=0.0196 0.0275 0.0164; visual mesh filename=link_0.0.obj
- link link_9.0: geometry collision box size=0.0196 0.0275 0.054; visual mesh filename=link_1.0.obj
